Commit message: chore: change urdf world name to base_footprint

File: src/axis_camera/urdf/axis_camera.xacro.urdf (robot description, URDF)
Before this commit: robot axis_camera, 5 links, 4 joints
Links:
- removed link world
- added link base_footprint
Joints:
- removed joint world_to_chassis
- added joint base_footprint_to_chassis: type fixed, parent base_footprint, child chassis, origin xyz=0 0 2 rpy=0 0 0

Commit message: chore: update axis_camera codes

File: src/axis_camera/urdf/axis_camera.xacro.urdf (robot description, URDF)
Before this commit: robot axis_camera, 5 links, 4 joints
Links:
- removed link base_footprint
- removed link chassis
- added link wall_link, mass 1
Joints:
- removed joint base_footprint_to_chassis
- removed joint chassis_to_pan
- added joint wall_to_pan: type revolute, parent wall_link, child pan_link, origin xyz=0.0 0.0 0.0, axis 0 0 1, limit lower=-600.28 upper=600.28 effort=100000 velocity=30
- joint tilt_to_camera: origin xyz=0.05 0 0 rpy=0 0 0 -> xyz=0.05 0 0 rpy=-1.5707963 0 -1.5707963; type revolute -> fixed
